File: unittests/eagleimport/testproject.brd (EAGLE design)
At the start: 100 x 80 mm, 4 parts, among them U1 TESTDEVICE, U2 TESTDEVICE, U3 TESTDEVICE, U4 TESTDEVICE

Commit message: Add buses to Eagle test project
Parts:
- added SV1, SV2: (no value), con-lsta:FE08
Connections:
- new net BUSA: SV1.2, SV2.2
- new net BUSB: SV1.1, SV2.1
- new net DATA0: SV1.6, SV1.8, SV2.6, SV2.8
- new net DATA1: SV1.5, SV1.7, SV2.5, SV2.7
Changed lines of the file:
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@@
 <?xml version="1.0" encoding="utf-8"?>
 <!DOCTYPE eagle SYSTEM "eagle.dtd">
-<eagle version="9.6.0">
+<eagle version="9.6.2">
 <drawing>
 <settings>
@@
 <attribute name="VALUE" x="71.764796875" y="32.54825" locked="yes" size="1.27" layer="28" font="vector" rot="MR5"/>
 </element>
+<element name="SV1" library="con-lsta" library_urn="urn:adsk.eagle:library:161" package="FE08" package3d_urn="urn:adsk.eagle:package:8194/1" value="" x="10.16" y="-3.81" smashed="yes">
+<attribute name="MF" value="" x="10.16" y="-3.81" size="1.778" layer="27" display="off"/>
+<attribute name="MPN" value="" x="10.16" y="-3.81" size="1.778" layer="27" display="off"/>
+<attribute name="NAME" x="3.81" y="-2.159" size="1.27" layer="25" ratio="10"/>
+<attribute name="OC_FARNELL" value="unknown" x="10.16" y="-3.81" size="1.778" layer="27" display="off"/>
+<attribute name="OC_NEWARK" value="unknown" x="10.16" y="-3.81" size="1.778" layer="27" display="off"/>
+<attribute name="POPULARITY" value="10" x="10.16" y="-3.81" size="1.778" layer="27" display="off"/>
+<attribute name="VALUE" x="0" y="-6.731" size="1.27" layer="27" ratio="10"/>
+</element>
+<element name="SV2" library="con-lsta" library_urn="urn:adsk.eagle:library:161" package="FE08" package3d_urn="urn:adsk.eagle:package:8194/1" value="" x="10.16" y="-8.89" smashed="yes">
+<attribute name="MF" value="" x="10.16" y="-8.89" size="1.778" layer="27" display="off"/>
+<attribute name="MPN" value="" x="10.16" y="-8.89" size="1.778" layer="27" display="off"/>
+<attribute name="NAME" x="3.81" y="-7.239" size="1.27" layer="25" ratio="10"/>
+<attribute name="OC_FARNELL" value="unknown" x="10.16" y="-8.89" size="1.778" layer="27" display="off"/>
+<attribute name="OC_NEWARK" value="unknown" x="10.16" y="-8.89" size="1.778" layer="27" display="off"/>
+<attribute name="POPULARITY" value="10" x="10.16" y="-8.89" size="1.778" layer="27" display="off"/>
+<attribute name="VALUE" x="0" y="-11.811" size="1.27" layer="27" ratio="10"/>
+</element>
 </elements>
 <signals>
@@
 <via x="46.99" y="39.37" extent="1-16" drill="0.35" diameter="1.27"/>
 </signal>
+<signal name="DATA0">
+<contactref element="SV1" pad="8"/>
+<contactref element="SV1" pad="6"/>
+<contactref element="SV2" pad="8"/>
+<contactref element="SV2" pad="6"/>
+<wire x1="13.97" y1="-3.81" x2="19.05" y2="-3.81" width="0" layer="19" extent="1-1"/>
+<wire x1="19.05" y1="-8.89" x2="19.05" y2="-3.81" width="0" layer="19" extent="1-1"/>
+<wire x1="13.97" y1="-8.89" x2="13.97" y2="-3.81" width="0" layer="19" extent="1-1"/>
+</signal>
+<signal name="DATA1">
+<contactref element="SV1" pad="7"/>
+<contactref element="SV1" pad="5"/>
+<contactref element="SV2" pad="7"/>
+<contactref element="SV2" pad="5"/>
+<wire x1="11.43" y1="-3.81" x2="16.51" y2="-3.81" width="0" layer="19" extent="1-1"/>
+<wire x1="16.51" y1="-8.89" x2="16.51" y2="-3.81" width="0" layer="19" extent="1-1"/>
+<wire x1="11.43" y1="-8.89" x2="11.43" y2="-3.81" width="0" layer="19" extent="1-1"/>
+</signal>
+<signal name="BUSB">
+<contactref element="SV1" pad="1"/>
+<contactref element="SV2" pad="1"/>
+<wire x1="1.27" y1="-3.81" x2="1.27" y2="-8.89" width="0" layer="19" extent="1-1"/>
+</signal>
+<signal name="BUSA">
+<contactref element="SV1" pad="2"/>
+<contactref element="SV2" pad="2"/>
+<wire x1="3.81" y1="-3.81" x2="3.81" y2="-8.89" width="0" layer="19" extent="1-1"/>
+</signal>
 </signals>
 <mfgpreviewcolors>
@@
 </board>
 </drawing>
+<compatibility>
+<note version="8.2" severity="warning">
+Since Version 8.2, EAGLE supports online libraries. The ids
+of those online libraries will not be understood (or retained)
+with this version.
+</note>
+<note version="8.3" severity="warning">
+Since Version 8.3, EAGLE supports URNs for individual library
+assets (packages, symbols, and devices). The URNs of those assets
+will not be understood (or retained) with this version.
+</note>
+<note version="8.3" severity="warning">
+Since Version 8.3, EAGLE supports the association of 3D packages
+with devices in libraries, schematics, and board files. Those 3D
+packages will not be understood (or retained) with this version.
+</note>
+</compatibility>
 </eagle>
